Commit message: test

File: urdf/ur.urdf.xacro (robot description, xacro)
@@ -54,5 +54,6 @@
    <xacro:property name="is_sim_ignition" value="$(arg sim_ignition)"/>
    <!-- create link fixed to the "world" -->
-   <link name="world" />
+   <link name="worldaaaa" />
+<link>
    <xacro:if value="${is_sim_gazebo or is_sim_ignition}">
      <link name="ground_plane">
